File: TIGER PCB Ver 0.2/TIGER Ver 0.2.kicad_sch (KiCad schematic)
At the start: 49 parts, among them J1 USB4105-GF-A, J2 Servo 2 Connector, J3 Servo 1 Connector, J4 Servo 3 Connector, J5 Servo 4 Connector, J7 MSD-4-A, J8 GPIO_R, J9 GPIO_L, SW1 SW_RESET, SW2 SW_RESET, U1 ESP32-S3-WROOM-1, U2 MPU-6050, U3 MPL3115A2, U4 AMS1117-3.3, U5 AMS1117-5.0, U6 USBLC6-2SC6, U7 Battery Socket

Commit message: Again
Parts:
- removed C14, C15: 100nF, Capacitor_SMD:C_0603_1608Metric, symbol Device:C
- removed D2: 5V LED, LED_SMD:LED_0603_1608Metric, symbol Device:LED
- removed R1: 5k1, Resistor_SMD:R_0603_1608Metric, symbol Device:R
- removed U2: MPU-6050, Sensor_Motion:InvenSense_QFN-24_4x4mm_P0.5mm, symbol Sensor_Motion:MPU-6050
- removed U6: USBLC6-2SC6, Package_TO_SOT_SMD:SOT-23-6, symbol Power_Protection:USBLC6-2SC6
- removed U7: Battery Socket, XT30UPB-M:XT30UPB-M, symbol XT30UPB-M:XT30UPB-M
- added D3: D+ LED, LED_SMD:LED_0603_1608Metric, symbol Device:LED
- added D4: D- LED, LED_SMD:LED_0603_1608Metric, symbol Device:LED
- added J10: Battery Connector, symbol Connector_Generic:Conn_01x02
- added J6: Conn_01x01_Pin, Connector_PinHeader_2.54mm:PinHeader_1x01_P2.54mm_Horizontal, symbol Connector:Conn_01x01_Pin
- added R12, R13: 5k1, Resistor_SMD:R_0603_1608Metric, symbol Device:R
- added U2: BMI270, .Custom Footprints:XDCR_BMI270, symbol BMI270:BMI270
- C13: value 2.2nF -> 100nF
- J1: footprint USB4105_GF_A:GCT_USB4105-GF-A -> .Custom Footprints:GCT_USB4105-GF-A
- J7: footprint MSD_4_A:CUI_MSD-4-A -> .Custom Footprints:CUI_MSD-4-A
Connections:
- net RAW_D+ is gone; now on net D+: J1.A6 (DP1), J1.B6 (DP2)
- net RAW_D- is gone; now on net D-: J1.A7 (DN1), J1.B7 (DN2)
- net +3V3: now also C13.1, C3.2, U2.12 (CSB), U2.5 (VDDIO), U2.8 (VDD); no longer C3.1
- net +BATT: now also J10.2 (Pin_2), J6.1 (Pin_1)
- net D+: now also R12.2
- net D-: now also R13.2
- net GND: now also C3.1, D3.1 (K), D4.1 (K), J10.1 (Pin_1), U2.1 (SDO), U2.6 (GNDIO), U2.7 (GND); no longer C3.2
- net I2C SCL: now also U2.13 (SCX)
- net I2C SDA: now also U2.14 (SDX)
- new net: D4.2 (A), R13.1
- new net: D3.2 (A), R12.1
- no-connect marks 10 -> 13
Other:
- note added: "BMI270"
- note removed: "10k pullup resistors for data lines Maybe don't need?"
- note removed: "I don't think SD Card wiring is correct but idk what else to put, I followed adafruit metro design"
- note removed: "I2C stuff is in the right place right?"
- note removed: "Is Power stuff fine? If the battery voltage is less than 12v then the LDO's should be fine right"
- note removed: "MPU-6050"
- note removed: "Most of this stuff should be fine since I copied it directly from ESP devboard schematics"

Commit message: lalala
Parts:
- removed J6: Conn_01x01_Pin, Connector_PinHeader_2.54mm:PinHeader_1x01_P2.54mm_Horizontal, symbol Connector:Conn_01x01_Pin
- J10: footprint (none) -> .Custom Footprints:Battery Connector
Connections:
- net +BATT: now also J8.22 (Pin_22)
- net GND: no longer J8.22 (Pin_22)
Changed lines of the file:
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@@
 	)
 	(symbol
-		(lib_id "Connector:Conn_01x01_Pin")
-		(at 132.08 204.47 0)
-		(unit 1)
-		(exclude_from_sim no)
-		(in_bom yes)
-		(on_board yes)
-		(dnp no)
-		(fields_autoplaced yes)
-		(property "Reference" "J6"
-			(at 132.715 199.39 0)
-			(effects
-				(font
-					(size 1.27 1.27)
-				)
-			)
-		)
-		(property "Value" "Conn_01x01_Pin"
-			(at 132.715 201.93 0)
-			(effects
-				(font
-					(size 1.27 1.27)
-				)
-			)
-		)
-		(property "Footprint" "Connector_PinHeader_2.54mm:PinHeader_1x01_P2.54mm_Horizontal"
-			(at 132.08 204.47 0)
-			(effects
-				(font
-					(size 1.27 1.27)
-				)
-				(hide yes)
-			)
-		)
-		(property "Datasheet" "~"
-			(at 132.08 204.47 0)
-			(effects
-				(font
-					(size 1.27 1.27)
-				)
-				(hide yes)
-			)
-		)
-		(property "Description" "Generic connector, single row, 01x01, script generated"
-			(at 132.08 204.47 0)
-			(effects
-				(font
-					(size 1.27 1.27)
-				)
-				(hide yes)
-			)
-		)
-		(pin "1"
-		)
-		(instances
-			(project ""
-				(path "/f0d0a6f4-8d43-4882-9cb7-06a2a1008823"
-					(reference "J6")
-					(unit 1)
-				)
-			)
-		)
-	)
-	(symbol
 		(lib_id "Connector:Conn_01x22_Pin")
 		(at 204.47 184.15 0)
@@
 			)
 		)
-		(property "Footprint" ""
+		(property "Footprint" ".Custom Footprints:Battery Connector"
 			(at 160.02 204.47 0)
 			(effects
@@
 	)
 	(symbol
-		(lib_id "power:GND")
-		(at 209.55 212.09 90)
-		(unit 1)
-		(exclude_from_sim no)
-		(in_bom yes)
-		(on_board yes)
-		(dnp no)
-		(fields_autoplaced yes)
-		(property "Reference" "#PWR051"
-			(at 215.9 212.09 0)
-			(effects
-				(font
-					(size 1.27 1.27)
-				)
-				(hide yes)
-			)
-		)
-		(property "Value" "GND"
-			(at 213.36 212.0899 90)
-			(effects
-				(font
-					(size 1.27 1.27)
-				)
-				(justify right)
-			)
-		)
-		(property "Footprint" ""
-			(at 209.55 212.09 0)
-			(effects
-				(font
-					(size 1.27 1.27)
-				)
-				(hide yes)
-			)
-		)
-		(property "Datasheet" ""
-			(at 209.55 212.09 0)
-			(effects
-				(font
-					(size 1.27 1.27)
-				)
-				(hide yes)
-			)
-		)
-		(property "Description" "Power symbol creates a global label with name \"GND\" , ground"
-			(at 209.55 212.09 0)
-			(effects
-				(font
-					(size 1.27 1.27)
-				)
-				(hide yes)
-			)
-		)
-		(pin "1"
-		)
-		(instances
-			(project "Rockets"
-				(path "/f0d0a6f4-8d43-4882-9cb7-06a2a1008823"
-					(reference "#PWR051")
-					(unit 1)
-				)
-			)
-		)
-	)
-	(symbol
 		(lib_id "Device:R")
 		(at 313.69 143.51 90)
@@
 	(symbol
 		(lib_id "power:+BATT")
-		(at 137.16 204.47 270)
+		(at 209.55 212.09 270)
 		(unit 1)
 		(exclude_from_sim no)
@@
 		(fields_autoplaced yes)
 		(property "Reference" "#PWR07"
-			(at 133.35 204.47 0)
+			(at 205.74 212.09 0)
 			(effects
 				(font
@@
 		)
 		(property "Value" "+BATT"
-			(at 140.97 204.4701 90)
+			(at 213.36 212.0901 90)
 			(effects
 				(font
@@
 		)
 		(property "Footprint" ""
-			(at 137.16 204.47 0)
+			(at 209.55 212.09 0)
 			(effects
 				(font
@@
 		)
 		(property "Datasheet" ""
-			(at 137.16 204.47 0)
+			(at 209.55 212.09 0)
 			(effects
 				(font
@@
 		)
 		(property "Description" "Power symbol creates a global label with name \"+BATT\""
-			(at 137.16 204.47 0)
+			(at 209.55 212.09 0)
 			(effects
 				(font

Commit message: More progress
Parts:
- removed D4: D- LED, LED_SMD:LED_0603_1608Metric, symbol Device:LED
- removed R13: 5k1, Resistor_SMD:R_0603_1608Metric, symbol Device:R
- added D2: D+ LED, LED_SMD:LED_0603_1608Metric, symbol Device:LED
- added R1: 5k1, Resistor_SMD:R_0603_1608Metric, symbol Device:R
- D1: value 3.3V LED -> D- LED
- D3: value D+ LED -> 3v3 LED
- renumbered C5 to C1, C18 to C10, C19 to C11, C2 to C12, C9 to C13, C4 to C14, C1 to C15, C3 to C16, C13 to C17, C10 to C2, C11 to C3, C8 to C4, C12 to C5, C16 to C8, C17 to C9, J3 to J2, J4 to J3, J2 to J4, J10 to J6, J9 to J7, J7 to J9, R8 to R10, R7 to R12, R12 to R2, R6 to R3, R9 to R6, R3 to R7, R2 to R8, R10 to R9, U4 to U1, U1 to U2, U5 to U3, U3 to U4, U2 to U5
Connections:
- net D-: now also R1.2
- net GND: now also D2.1 (K)
- net at D1.2 (A): now also R1.1; no longer R6.2
- net at D3.2 (A): now also R6.2; no longer R2.1
- new net: D2.2 (A), R2.1

Commit message: Layout almost done
Parts:
- removed J7: GPIO_L, Connector_PinSocket_2.54mm:PinSocket_1x22_P2.54mm_Vertical, symbol Connector:Conn_01x22_Pin
- removed J8: GPIO_R, Connector_PinSocket_2.54mm:PinSocket_1x22_P2.54mm_Vertical, symbol Connector:Conn_01x22_Pin
- added H1, H2, H3, H4: MountingHole, MountingHole:MountingHole_3.2mm_M3, symbol Mechanical:MountingHole
- added J10, J11: Conn_01x09_Socket, Connector_PinSocket_2.54mm:PinSocket_1x09_P2.54mm_Vertical, symbol Connector:Conn_01x09_Socket
- J2: value Servo 1 Connector -> Servo 1
- J3: value Servo 3 Connector -> Servo 3
- J4: value Servo 2 Connector -> Servo 2
- J5: value Servo 4 Connector -> Servo 4
Connections:
- net +3V3: now also J11.1 (Pin_1)
- net +5V: now also J11.2 (Pin_2)
- net +BATT: now also J11.3 (Pin_3)
- net D+: now also J11.9 (Pin_9)
- net D-: now also J11.8 (Pin_8)
- net GND: now also J10.9 (Pin_9)
- net I2C SCL: now also J10.7 (Pin_7)
- net I2C SDA: now also J10.8 (Pin_8)
- net RX: now also J10.1 (Pin_1)
- net SERVO_1: now also J10.3 (Pin_3)
- net SERVO_2: now also J10.4 (Pin_4)
- net SERVO_3: now also J10.5 (Pin_5)
- net SERVO_4: now also J10.6 (Pin_6)
- net SPI_CS: now also J11.4 (Pin_4)
- net SPI_MISO: now also J11.7 (Pin_7)
- net SPI_MOSI: now also J11.5 (Pin_5)
- net SPI_SCK: now also J11.6 (Pin_6)
- net TX: now also J10.2 (Pin_2)
