File: TIGER PCB Ver 0.2/TIGER Ver 0.2.kicad_pcb (KiCad board)
At the start: 2 copper layers, 52.2 x 60.8 mm, 51 parts, among them J1 USB4105-GF-A, J2 Servo 2 Connector, J3 Servo 1 Connector, J4 Servo 3 Connector, J5 Servo 4 Connector, J7 MSD-4-A, J8 GPIO_R, J9 GPIO_L, SW1 SW_RESET, SW2 SW_RESET, U1 ESP32-S3-WROOM-1, U2 MPU-6050, U3 MPL3115A2, U4 AMS1117-3.3, U5 AMS1117-5.0, U6 USBLC6-2SC6, U7 Battery Socket

Commit message: Again
Parts:
- removed 3v3: 3.3V LED, LED_SMD:LED_0603_1608Metric
- removed 5v: 5V LED, LED_SMD:LED_0603_1608Metric
- removed the C13 at (133.8, 64.5)
- removed the C3 at (136.8, 66.8)
- removed the G*** at (117.4, 68.8)
- removed the U2 at (133.0, 68.5)
- removed U7: Battery Socket, XT30UPB-M:XT30UPB-M
- added C13: 2.2nF, Capacitor_SMD:C_0603_1608Metric, F.Cu at (119.9, 95.1)
- added C13: 100nF, Capacitor_SMD:C_0603_1608Metric, F.Cu at (204.1, 84.2)
- added C3: 100nF, Capacitor_SMD:C_0603_1608Metric, F.Cu at (204.1, 81.7)
- added C3: 100nF, Capacitor_SMD:C_0603_1608Metric, F.Cu at (111.9, 100.1)
- added D1: 3.3V LED, LED_SMD:LED_0603_1608Metric, F.Cu at (164.2, 95.2)
- added D2: 5V LED, LED_SMD:LED_0603_1608Metric, F.Cu at (164.2, 97.8)
- added D3: D+ LED, LED_SMD:LED_0603_1608Metric, F.Cu at (208.2, 81.8)
- added D4: D- LED, LED_SMD:LED_0603_1608Metric, F.Cu at (208.2, 84.4)
- added J6: Conn_01x01_Pin, Connector_PinHeader_2.54mm:PinHeader_1x01_P2.54mm_Horizontal, F.Cu at (204.4, 78.2)
- added R12: 5k1, Resistor_SMD:R_0603_1608Metric, F.Cu at (204.1, 86.8)
- added R13: 5k1, Resistor_SMD:R_0603_1608Metric, F.Cu at (204.1, 89.3)
- added U2: MPU-6050, Sensor_Motion:InvenSense_QFN-24_4x4mm_P0.5mm, F.Cu at (159.0, 97.0)
- added U2: BMI270, .Custom Footprints:XDCR_BMI270, F.Cu at (212.8, 82.5)
- J1: footprint USB4105_GF_A:GCT_USB4105-GF-A -> .Custom Footprints:GCT_USB4105-GF-A
- J7: footprint MSD_4_A:CUI_MSD-4-A -> .Custom Footprints:CUI_MSD-4-A
- moved J7 87.6 mm to (193.0, 75.6)
- moved J1 78.5 mm to (207.7, 72.5)
- moved J5 65.8 mm to (161.9, 74.0), turned to 0 degrees
- moved C6 62.8 mm to (111.9, 107.7), turned to 0 degrees
- moved J4 60.5 mm to (161.9, 67.4), turned to 0 degrees
- moved R5 55.5 mm to (123.9, 107.7), turned to 0 degrees
- moved R2 47.7 mm to (123.9, 100.1), turned to 0 degrees
- moved G*** 45.8 mm to (72.2, 68.2)
- moved C7 45.2 mm to (115.9, 95.1), turned to 0 degrees
- moved SW1 43.4 mm to (132.0, 95.9)
- moved R3 42.6 mm to (123.9, 102.7), turned to 0 degrees
- moved U3 41.0 mm to (153.3, 97.2)
- moved J8 39.0 mm to (103.0, 53.9)
- moved U6 37.8 mm to (158.4, 102.6)
- moved C8 37.6 mm to (115.9, 97.6), turned to 0 degrees
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Connections:
- J1 pad A6: RAW_D+ -> D+
- J1 pad A7: RAW_D- -> D-
- J1 pad B6: RAW_D+ -> D+
- J1 pad B7: RAW_D- -> D-
Routing:
- net GND: track 211.9 -> 0.00 mm, vias 37 -> 0
- net ESP 3v3: track 176.3 -> 0.00 mm, vias 12 -> 0
- net +5V: track 139.2 -> 0.00 mm, vias 8 -> 0
- net SERVO_2: track 99.6 -> 0.00 mm, vias 4 -> 0
- net SPI_SCK: track 79.8 -> 0.00 mm, vias 5 -> 0
- net SERVO_1: track 79.0 -> 0.00 mm, vias 4 -> 0
- net SPI_MISO: track 78.7 -> 0.00 mm, vias 11 -> 0
- net SPI_MOSI: track 75.4 -> 0.00 mm, vias 6 -> 0
- net BOOT: track 69.6 -> 0.00 mm, vias 5 -> 0
- net CHIP_PU: track 63.8 -> 0.00 mm, vias 2 -> 0
- net D-: track 63.2 -> 0.00 mm, vias 6 -> 0
- net IO_37: track 60.1 -> 0.00 mm, vias 2 -> 0
- net D+: track 59.9 -> 0.00 mm, vias 6 -> 0
- net SERVO_4: track 53.4 -> 0.00 mm, vias 3 -> 0
- net IO_38: track 52.6 -> 0.00 mm
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- removed copper zone on B.Cu, net GND
Other:
- board outline removed
- board text removed: "0"
- board text removed: "1"
- board text removed: "10"
- board text removed: "11"
- board text removed: "12"
- board text removed: "13"
- board text removed: "14"
- board text removed: "15"
- board text removed: "16"
- board text removed: "17"
- board text removed: "18"
- board text removed: "2"
- board text removed: "21"
- board text removed: "3"
- board text removed: "35"
- board text removed: "36"
- board text removed: "37"
- board text removed: "38"
- board text removed: "39"
- board text removed: "3v3"
- board text removed: "4"
- board text removed: "40"
- board text removed: "41"
- board text removed: "42"
- board text removed: "45"
- board text removed: "46"
- board text removed: "47"
- board text removed: "48"
- board text removed: "5"
- board text removed: "5V"
- board text removed: "7"
- board text removed: "8"
- board text removed: "9"
- board text removed: "D+"
- board text removed: "D-"
- board text removed: "GND"
- board text removed: "Pinouts follow ESP32 S3 Dev Kit C, the Right side is the same, Left side is flipped upside down"
- board text removed: "RST"
- board text removed: "RX"
- board text removed: "T.I.G.E.R Ver 0.1"
- board text removed: "TX"

Commit message: lalala
Parts:
- removed the C13 at (119.9, 95.1)
- removed the C13 at (204.1, 84.2)
- removed C14, C15: 100nF, Capacitor_SMD:C_0603_1608Metric
- removed the C3 at (204.1, 81.7)
- removed the C3 at (111.9, 100.1)
- removed D2: 5V LED, LED_SMD:LED_0603_1608Metric
- removed G***: LOGO, Custom Footprints:PHS Tigers Logo
- removed J6: Conn_01x01_Pin, Connector_PinHeader_2.54mm:PinHeader_1x01_P2.54mm_Horizontal
- removed R1: 5k1, Resistor_SMD:R_0603_1608Metric
- removed SW1, SW2: SW_RESET, Button_Switch_THT:SW_PUSH_6mm
- removed the U2 at (159.0, 97.0)
- removed the U2 at (212.8, 82.5)
- removed U4: AMS1117-3.3, Package_TO_SOT_SMD:SOT-223-3_TabPin2
- removed U5: AMS1117-5.0, Package_TO_SOT_SMD:SOT-223-3_TabPin2
- removed U6: USBLC6-2SC6, Package_TO_SOT_SMD:SOT-23-6
- added 3v3  : AMS1117-3.3, Package_TO_SOT_SMD:SOT-223-3_TabPin2, F.Cu at (124.2, 72.2)
- added 5v: AMS1117-5.0, Package_TO_SOT_SMD:SOT-223-3_TabPin2, F.Cu at (80.0, 83.0)
- added BOOT: SW_RESET, Button_Switch_THT:SW_PUSH_6mm, F.Cu at (101.3, 68.1)
- added C13: 100nF, Capacitor_SMD:C_0603_1608Metric, F.Cu at (116.5, 156.0)
- added C3: 100nF, Capacitor_SMD:C_0603_1608Metric, B.Cu at (127.2, 75.8)
- added J10: Battery Connector, .Custom Footprints:Battery Connector, F.Cu at (119.5, 97.2)
- added REF**: MountingHole_4.3mm_M4_Pad_Via, MountingHole:MountingHole_4.3mm_M4_Pad_Via, F.Cu at (148.5, 105.5)
- added REF**: MountingHole_4.3mm_M4_Pad_Via, MountingHole:MountingHole_4.3mm_M4_Pad_Via, F.Cu at (86.5, 47.8)
- added REF**: MountingHole_4.3mm_M4_Pad_Via, MountingHole:MountingHole_4.3mm_M4_Pad_Via, F.Cu at (149.8, 47.8)
- added REF**: MountingHole_4.3mm_M4_Pad_Via, MountingHole:MountingHole_4.3mm_M4_Pad_Via, F.Cu at (86.0, 106.8)
- added RESET: SW_RESET, Button_Switch_THT:SW_PUSH_6mm, F.Cu at (130.4, 72.2)
- added U2: BMI270, .Custom Footprints:XDCR_BMI270, F.Cu at (118.0, 68.5)
- C1, C2, J7: moved to B.Cu
- J2: value Servo 2 Connector -> Servo 2
- J3: value Servo 1 Connector -> Servo 1
- J4: value Servo 3 Connector -> Servo 3
- J5: value Servo 4 Connector -> Servo 4
- moved R12 103.9 mm to (124.5, 153.5)
- moved R13 103.9 mm to (124.5, 156.0)
- moved J7 89.1 mm to (104.8, 87.8), turned to 180 degrees
- moved D3 81.7 mm to (126.5, 82.8)
- moved J1 76.5 mm to (133.2, 90.0)
- moved D4 74.5 mm to (133.8, 80.0)
- moved C7 66.0 mm to (112.5, 161.0)
- moved C8 66.0 mm to (112.5, 163.5)
- moved R7 63.8 mm to (120.5, 161.0)
- moved R8 63.8 mm to (120.5, 163.5)
- moved R6 63.8 mm to (120.5, 158.5)
- moved J4 62.5 mm to (101.9, 49.8), turned to -45 degrees
- moved J5 61.7 mm to (101.9, 59.7), turned to -45 degrees
- moved C17 56.0 mm to (116.5, 161.0)
- moved C18 56.0 mm to (116.5, 163.5)
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Connections:
- J8 pad 22: GND -> +BATT

Commit message: More progress
Parts:
- removed D4: D- LED, LED_SMD:LED_0603_1608Metric
- removed R13: 5k1, Resistor_SMD:R_0603_1608Metric
- removed the REF** at (148.5, 105.5)
- removed the REF** at (86.5, 47.8)
- removed the REF** at (149.8, 47.8)
- removed the REF** at (86.0, 106.8)
- added D2: D+ LED, LED_SMD:LED_0603_1608Metric, F.Cu at (129.2, 102.9)
- added R1: 5k1, Resistor_SMD:R_0603_1608Metric, F.Cu at (133.2, 100.2)
- added REF**: MountingHole_4.3mm_M4_Pad_Via, MountingHole:MountingHole_4.3mm_M4_Pad_Via, F.Cu at (150.5, 47.2)
- added REF**: MountingHole_4.3mm_M4_Pad_Via, MountingHole:MountingHole_4.3mm_M4_Pad_Via, F.Cu at (85.2, 106.8)
- added REF**: MountingHole_4.3mm_M4_Pad_Via, MountingHole:MountingHole_4.3mm_M4_Pad_Via, F.Cu at (150.8, 106.2)
- added REF**: MountingHole_4.3mm_M4_Pad_Via, MountingHole:MountingHole_4.3mm_M4_Pad_Via, F.Cu at (85.2, 46.0)
- C1: renamed from C5; moved to B.Cu
- D1: value 3.3V LED -> D- LED
- D3: value D+ LED -> 3v3 LED
- J2: renamed from J3; value Servo 1 -> Servo 1 Connector
- J3: renamed from J4; value Servo 3 -> Servo 3 Connector
- J4: renamed from J2; value Servo 2 -> Servo 2 Connector
- J5: value Servo 4 -> Servo 4 Connector
- U1: renamed from 3v3  
- moved C1 84.9 mm to (126.5, 72.2), turned to -90 degrees
- moved U3 33.8 mm to (112.0, 72.0)
- moved D3 22.9 mm to (129.2, 105.5)
- moved D1 17.9 mm to (129.2, 100.3)
- renumbered C18 to C10, C19 to C11, C2 to C12, C9 to C13, C4 to C14, C1 to C15, C3 to C16, C13 to C17, C10 to C2, C11 to C3, C8 to C4, C12 to C5, C16 to C8, C17 to C9, J10 to J6, J9 to J7, J7 to J9, R8 to R10, R7 to R12, R12 to R2, R6 to R3, R9 to R6, R3 to R7, R2 to R8, R10 to R9, BOOT to SW1, RESET to SW2, U1 to U2, 5v to U3, U3 to U4, U2 to U5
Connections:
- R2 pad 1: Net-(D3-A) -> Net-(D2-A)
- R6 pad 2: Net-(D1-A) -> Net-(D3-A)

Commit message: Layout almost done
Parts:
- removed J7: GPIO_L, Connector_PinSocket_2.54mm:PinSocket_1x22_P2.54mm_Vertical
- removed J8: GPIO_R, Connector_PinSocket_2.54mm:PinSocket_1x22_P2.54mm_Vertical
- removed REF** (x4): MountingHole_4.3mm_M4_Pad_Via, MountingHole:MountingHole_4.3mm_M4_Pad_Via
- added H1: MountingHole, MountingHole:MountingHole_3.2mm_M3, F.Cu at (163.8, 72.0)
- added H2: MountingHole, MountingHole:MountingHole_3.2mm_M3, F.Cu at (115.2, 71.8)
- added H3: MountingHole, MountingHole:MountingHole_3.2mm_M3, F.Cu at (114.2, 119.0)
- added H4: MountingHole, MountingHole:MountingHole_3.2mm_M3, F.Cu at (163.2, 119.2)
- added J10: Conn_01x09_Socket, Connector_PinSocket_2.54mm:PinSocket_1x09_P2.54mm_Vertical, F.Cu at (164.0, 84.5)
- added J11: Conn_01x09_Socket, Connector_PinSocket_2.54mm:PinSocket_1x09_P2.54mm_Vertical, F.Cu at (115.8, 84.7)
- C10, C11, C17, C2, C3, C5, C6, C7, C8, C9, R1, R10, R11, R12, R2, R3, R4, R5, R6, R7, R8, R9: moved to B.Cu
- J2: value Servo 1 Connector -> Servo 1
- J3: value Servo 3 Connector -> Servo 3
- J4: value Servo 2 Connector -> Servo 2
- J5: value Servo 4 Connector -> Servo 4
- moved C7 98.4 mm to (146.2, 68.6), turned to 90 degrees
- moved C6 92.3 mm to (133.2, 68.6), turned to 90 degrees
- moved C4 90.2 mm to (158.4, 85.8), turned to 135 degrees
- moved R5 84.9 mm to (133.2, 72.1), turned to 90 degrees
- moved R8 80.3 mm to (146.2, 72.3), turned to 90 degrees
- moved C10 76.8 mm to (136.4, 89.3), turned to -90 degrees
- moved C17 72.0 mm to (139.7, 87.8)
- moved C9 69.4 mm to (131.9, 93.3), turned to 180 degrees
- moved C8 67.9 mm to (135.7, 93.3), turned to 180 degrees
- moved C5 66.2 mm to (144.2, 93.3), turned to 180 degrees
- moved C3 65.4 mm to (147.4, 93.3)
- moved C2 64.7 mm to (142.9, 89.4), turned to 90 degrees
- moved R10 61.5 mm to (141.5, 105.8)
- moved R3 60.8 mm to (153.4, 107.3)
- moved R7 60.0 mm to (140.9, 94.6), turned to -90 degrees
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Other:
- board outline added: 68.5 x 58.2 mm
- board text added: "Boot"
- board text added: "Reset"

Commit message: Finished Layout
Parts:
- added G***: LOGO, .Custom Footprints:PHS Tigers Logo, F.Cu at (142.9, 105.3)
- C13, C14, C4: moved to B.Cu
- J9: moved to F.Cu
- moved C4 23.5 mm to (140.0, 71.2), turned to 0 degrees
- moved C14 22.7 mm to (158.8, 85.8), turned to 135 degrees
- moved R11 12.5 mm to (129.3, 106.4)
- moved R9 12.5 mm to (125.8, 106.4)
- moved R10 8.28 mm to (133.2, 106.5), turned to 180 degrees
- moved R12 8.04 mm to (146.0, 106.5), turned to 0 degrees
- moved H3 7.32 mm to (115.2, 111.8)
- moved H4 7.32 mm to (164.2, 112.0)
- moved J6 6.87 mm to (142.5, 118.4)
- moved J9 6.55 mm to (127.8, 109.7), turned to 0 degrees
- moved R4 5.02 mm to (153.5, 106.5)
- moved J1 4.75 mm to (154.8, 116.0)
- moved R3 3.80 mm to (149.8, 106.5)
- moved J10 2.83 mm to (164.2, 81.6)
- moved J11 2.61 mm to (115.0, 82.2)
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- renumbered D3 to VDD
Other:
- board size 68.5 x 58.2 mm -> 60.5 x 51.5 mm
- board text added: "3v3"
- board text added: "5v"
- board text added: "D+"
- board text added: "D-"
- board text added: "T.I.G.E.R Ver 0.2"
- board text added: "vBat"

Commit message: Ver 0.2 Completed
Parts:
- moved R7 14.7 mm to (142.5, 80.0), turned to 0 degrees
- moved R8 12.6 mm to (136.2, 80.0), turned to 180 degrees
- moved C4 6.30 mm to (146.2, 72.0), turned to 90 degrees
Routing:
- net ESP 3v3: track 0.00 -> 127.7 mm, vias 0 -> 5
- net I2C SDA: track 0.00 -> 105.0 mm, vias 0 -> 6
- net +5V: track 0.00 -> 95.9 mm, vias 0 -> 4
- net D-: track 0.00 -> 94.1 mm, vias 0 -> 2
- net +BATT: track 0.00 -> 83.2 mm, vias 0 -> 2
- net D+: track 0.00 -> 76.1 mm, vias 0 -> 2
- net SERVO_3: track 0.00 -> 75.7 mm, vias 0 -> 1
- net SPI_CS: track 0.00 -> 73.2 mm, vias 0 -> 2
- net SPI_MISO: track 0.00 -> 70.8 mm, vias 0 -> 1
- net I2C SCL: track 0.00 -> 59.5 mm, vias 0 -> 3
- net CHIP_PU: track 0.00 -> 56.8 mm, vias 0 -> 2
- net SERVO_4: track 0.00 -> 54.8 mm, vias 0 -> 2
- net SPI_SCK: track 0.00 -> 54.1 mm, vias 0 -> 2
- net SERVO_2: track 0.00 -> 49.7 mm, vias 0 -> 1
- net BOOT: track 0.00 -> 46.8 mm
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- added copper zone on B.Cu, net GND
Other:
- board text added: "10"
- board text added: "11"
- board text added: "12"
- board text added: "13"
- board text added: "35"
- board text added: "36"
- board text added: "4"
- board text added: "5"
- board text added: "6"
- board text added: "7"
- board text added: "GND"
- board text added: "RX"
- board text added: "TX"

Commit message: TIGER Ver 0.2 Final
Routing:
- net GND: track 45.0 -> 178.9 mm, vias 16 -> 35
- net +BATT: track 83.2 -> 84.3 mm
- net SERVO_3: track 75.7 -> 75.0 mm, vias 1 -> 3
